File: PC104 Cubesat Template/PC104 Cubesat Template.kicad_pcb (KiCad board)
At the start: 2 copper layers, 90.2 x 95.9 mm, 10 parts

Commit message: add tj bus specific pins
Connections:
- H1 pad 1: (no net) -> unconnected-(H1-Pad1)
- H1 pad 10: (no net) -> unconnected-(H1-Pad10)
- H1 pad 11: (no net) -> TX2/GP8
- H1 pad 12: (no net) -> unconnected-(H1-Pad12)
- H1 pad 13: (no net) -> GP15/A1/RX3
- H1 pad 14: (no net) -> unconnected-(H1-Pad14)
- H1 pad 15: (no net) -> unconnected-(H1-Pad15)
- H1 pad 16: (no net) -> unconnected-(H1-Pad16)
- H1 pad 17: (no net) -> GP21/A7/RX5
- H1 pad 18: (no net) -> unconnected-(H1-Pad18)
- H1 pad 19: (no net) -> unconnected-(H1-Pad19)
- H1 pad 2: (no net) -> unconnected-(H1-Pad2)
- H1 pad 20: (no net) -> unconnected-(H1-Pad20)
- H1 pad 21: (no net) -> unconnected-(H1-Pad21)
- H1 pad 22: (no net) -> unconnected-(H1-Pad22)
- H1 pad 23: (no net) -> unconnected-(H1-Pad23)
- H1 pad 24: (no net) -> unconnected-(H1-Pad24)
- H1 pad 25: (no net) -> unconnected-(H1-Pad25)
- H1 pad 26: (no net) -> unconnected-(H1-Pad26)
- H1 pad 27: (no net) -> unconnected-(H1-Pad27)
- H1 pad 28: (no net) -> unconnected-(H1-Pad28)
- H1 pad 29: (no net) -> unconnected-(H1-Pad29)
- H1 pad 3: (no net) -> unconnected-(H1-Pad3)
- H1 pad 30: (no net) -> unconnected-(H1-Pad30)
- H1 pad 31: (no net) -> unconnected-(H1-Pad31)
- H1 pad 32: (no net) -> unconnected-(H1-Pad32)
- H1 pad 33: (no net) -> unconnected-(H1-Pad33)
- H1 pad 34: (no net) -> unconnected-(H1-Pad34)
- H1 pad 35: (no net) -> unconnected-(H1-Pad35)
- H1 pad 36: (no net) -> unconnected-(H1-Pad36)
- H1 pad 37: (no net) -> unconnected-(H1-Pad37)
- H1 pad 38: (no net) -> unconnected-(H1-Pad38)
- H1 pad 39: (no net) -> unconnected-(H1-Pad39)
- H1 pad 4: (no net) -> unconnected-(H1-Pad4)
- H1 pad 40: (no net) -> unconnected-(H1-Pad40)
- H1 pad 41: (no net) -> unconnected-(H1-Pad41)
- H1 pad 42: (no net) -> unconnected-(H1-Pad42)
- H1 pad 43: (no net) -> unconnected-(H1-Pad43)
- H1 pad 44: (no net) -> unconnected-(H1-Pad44)
- H1 pad 45: (no net) -> unconnected-(H1-Pad45)
- H1 pad 46: (no net) -> CS/GP10
- H1 pad 47: (no net) -> unconnected-(H1-Pad47)
- H1 pad 48: (no net) -> CS/GP37
- H1 pad 49: (no net) -> unconnected-(H1-Pad49)
- H1 pad 5: (no net) -> unconnected-(H1-Pad5)
- H1 pad 50: (no net) -> CS/GP36
- H1 pad 51: (no net) -> unconnected-(H1-Pad51)
- H1 pad 52: (no net) -> unconnected-(H1-Pad52)
- H1 pad 6: (no net) -> unconnected-(H1-Pad6)
- H1 pad 7: (no net) -> TX1/GP1
- H1 pad 8: (no net) -> unconnected-(H1-Pad8)
- H1 pad 9: (no net) -> RX2/GP7
- H2 pad 1: (no net) -> unconnected-(H2-Pad1)
- H2 pad 10: (no net) -> SW2
- H2 pad 11: (no net) -> SW3
- H2 pad 12: (no net) -> SW4
- H2 pad 13: (no net) -> SW5
- H2 pad 14: (no net) -> SW6
- H2 pad 15: (no net) -> SW7
- H2 pad 16: (no net) -> SW8
- H2 pad 17: (no net) -> SW9
- H2 pad 18: (no net) -> SW10
- H2 pad 19: (no net) -> SW11
- H2 pad 2: (no net) -> unconnected-(H2-Pad2)
- H2 pad 20: (no net) -> SW12
- H2 pad 21: (no net) -> unconnected-(H2-Pad21)
- H2 pad 22: (no net) -> unconnected-(H2-Pad22)
- H2 pad 23: (no net) -> unconnected-(H2-Pad23)
- H2 pad 24: (no net) -> unconnected-(H2-Pad24)
- H2 pad 25: +5V -> unconnected-(H2-Pad25)
- H2 pad 26: +5V -> unconnected-(H2-Pad26)
- H2 pad 27: +3V3 -> unconnected-(H2-Pad27)
- H2 pad 28: +3V3 -> unconnected-(H2-Pad28)
- H2 pad 29: GND -> unconnected-(H2-Pad29)
- H2 pad 3: (no net) -> unconnected-(H2-Pad3)
- H2 pad 30: GND -> unconnected-(H2-Pad30)
- H2 pad 31: (no net) -> unconnected-(H2-Pad31)
- H2 pad 32: GND -> unconnected-(H2-Pad32)
- H2 pad 33: (no net) -> unconnected-(H2-Pad33)
- H2 pad 34: (no net) -> unconnected-(H2-Pad34)
- H2 pad 35: (no net) -> PCM_IN
- H2 pad 36: (no net) -> unconnected-(H2-Pad36)
- H2 pad 37: (no net) -> unconnected-(H2-Pad37)
- H2 pad 38: (no net) -> unconnected-(H2-Pad38)
- H2 pad 39: (no net) -> unconnected-(H2-Pad39)
- H2 pad 4: (no net) -> unconnected-(H2-Pad4)
- H2 pad 40: (no net) -> unconnected-(H2-Pad40)
- H2 pad 41: (no net) -> BCR_OUT
- H2 pad 42: (no net) -> unconnected-(H2-Pad42)
- H2 pad 43: (no net) -> BCR_OUT
- H2 pad 44: (no net) -> BCR_OUT
- H2 pad 45: +BATT -> unconnected-(H2-Pad45)
- H2 pad 46: +BATT -> unconnected-(H2-Pad46)
- H2 pad 47: (no net) -> unconnected-(H2-Pad47)
- H2 pad 48: (no net) -> unconnected-(H2-Pad48)
- H2 pad 49: (no net) -> unconnected-(H2-Pad49)
- H2 pad 5: (no net) -> unconnected-(H2-Pad5)
- H2 pad 50: (no net) -> unconnected-(H2-Pad50)
- H2 pad 51: (no net) -> unconnected-(H2-Pad51)
- H2 pad 52: (no net) -> unconnected-(H2-Pad52)
- H2 pad 6: (no net) -> unconnected-(H2-Pad6)
- H2 pad 7: (no net) -> unconnected-(H2-Pad7)
- H2 pad 8: (no net) -> unconnected-(H2-Pad8)
- H2 pad 9: (no net) -> SW1
